Commit message: Removed absolute path from epistemic.worldo and head.urdf.xacro

File: src/tiago/tiago_robot/tiago_description/urdf/head/head.urdf.xacro (robot description, xacro)
@@ -112,5 +112,5 @@
         <origin xyz="0 0 0" rpy="0 0 0" />
         <geometry>
-          <mesh filename="/home/afavier/new_exec_sim_ws/src/simulator/meshes/tiago_eyes.dae" scale="1 1 1"/>
+          <mesh filename="$(find simulator)/meshes/tiago_eyes.dae" scale="1 1 1"/>
         </geometry>
         <material name="Black" />
